Commit message: feat: Add custom launch scripts and controller configurations for right arm of Kinova Gen3
- Created my_right_gen3.launch.py for dynamic injection of gripper joint name prefix to avoid registration conflicts.
- Added recover_controllers.sh script for safely resetting right arm controllers after emergency stops.
- Introduced right_gripper_controller.yaml for configuring the Robotiq 2F-85 gripper parameters.
- Developed right_ros2_controllers.yaml to resolve namespace issues with controller parameters for the right arm.
- Implemented start_dual_gen3_cumotion.py for a streamlined dual-arm startup process with active polling for controller readiness.
- Added start_dual_gen3_real_alfred.py for a quick startup of the dual-arm system with joint limits and active polling.

File: ros2_kortex_ws/Kortex_ws/src/dual_arm_control_bringup/config/my_dual_gen3.urdf (robot description, URDF)
Before this commit: robot dual_gen3_with_gripper, 42 links, 41 joints
Links:
- link left_base_link: geometry collision mesh filename=package://kortex_description/arms/gen3/7dof/meshes/base_lin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 scale=1.15 1.15 1.15; visual mesh filename=package://kortex_description/arms/gen3/7dof/meshes/base_lin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
- link left_bracelet_link: geometry collision mesh filename=package://kortex_description/arms/gen3/7dof/meshes/bracelet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 scale=1.15 1.15 1.15; visual mesh filename=package://kortex_description/arms/gen3/7dof/meshes/bracelet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
- link left_forearm_link: geometry collision mesh filename=package://kortex_description/arms/gen3/7dof/meshes/forearm_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 scale=1.15 1.15 1.15; visual mesh filename=package://kortex_description/arms/gen3/7dof/meshes/forearm_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
- link left_half_arm_1_link: geometry collision mesh filename=package://kortex_description/arms/gen3/7dof/meshes/half_arm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 scale=1.15 1.15 1.15; visual mesh filename=package://kortex_description/arms/gen3/7dof/meshes/half_arm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
- link left_half_arm_2_link: geometry collision mesh filename=package://kortex_description/arms/gen3/7dof/meshes/half_arm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 scale=1.15 1.15 1.15; visual mesh filename=package://kortex_description/arms/gen3/7dof/meshes/half_arm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
- link left_robotiq_85_base_link: geometry collision mesh filename=package://dual_arm_control_bringup/config/robotiq_descripti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 scale=1.15 1.15 1.15; visual mesh filename=package://dual_arm_control_bringup/config/robotiq_descripti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
- link left_robotiq_85_left_finger_link: geometry collision mesh filename=package://dual_arm_control_bringup/config/robotiq_descripti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 scale=1.15 1.15 1.15; visual mesh filename=package://dual_arm_control_bringup/config/robotiq_descripti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
- link left_robotiq_85_left_finger_tip_link: geometry collision mesh filename=package://dual_arm_control_bringup/config/robotiq_descripti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 scale=1.15 1.15 1.15; visual mesh filename=package://dual_arm_control_bringup/config/robotiq_descripti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
- link left_robotiq_85_left_inner_knuckle_link: geometry collision mesh filename=package://dual_arm_control_bringup/config/robotiq_descripti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 scale=1.15 1.15 1.15; visual mesh filename=package://dual_arm_control_bringup/config/robotiq_descripti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
- link left_robotiq_85_left_knuckle_link: geometry collision mesh filename=package://dual_arm_control_bringup/config/robotiq_descripti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 scale=1.15 1.15 1.15; visual mesh filename=package://dual_arm_control_bringup/config/robotiq_descripti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
- link left_robotiq_85_right_finger_link: geometry collision mesh filename=package://dual_arm_control_bringup/config/robotiq_descripti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 scale=1.15 1.15 1.15; visual mesh filename=package://dual_arm_control_bringup/config/robotiq_descripti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
- link left_robotiq_85_right_finger_tip_link: geometry collision mesh filename=package://dual_arm_control_bringup/config/robotiq_descripti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 scale=1.15 1.15 1.15; visual mesh filename=package://dual_arm_control_bringup/config/robotiq_descripti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
- link left_robotiq_85_right_inner_knuckle_link: geometry collision mesh filename=package://dual_arm_control_bringup/config/robotiq_descripti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 scale=1.15 1.15 1.15; visual mesh filename=package://dual_arm_control_bringup/config/robotiq_descripti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
- link left_robotiq_85_right_knuckle_link: geometry collision mesh filename=package://dual_arm_control_bringup/config/robotiq_descripti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 scale=1.15 1.15 1.15; visual mesh filename=package://dual_arm_control_bringup/config/robotiq_descripti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
- link left_shoulder_link: geometry collision mesh filename=package://kortex_description/arms/gen3/7dof/meshes/shoulder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 scale=1.15 1.15 1.15; visual mesh filename=package://kortex_description/arms/gen3/7dof/meshes/shoulder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
- link left_spherical_wrist_1_link: geometry collision mesh filename=package://kortex_description/arms/gen3/7dof/meshes/spherica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 scale=1.15 1.15 1.15; visual mesh filename=package://kortex_description/arms/gen3/7dof/meshes/spherica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
- link left_spherical_wrist_2_link: geometry collision mesh filename=package://kortex_description/arms/gen3/7dof/meshes/spherica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 scale=1.15 1.15 1.15; visual mesh filename=package://kortex_description/arms/gen3/7dof/meshes/spherica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
- link right_base_link: geometry collision mesh filename=package://kortex_description/arms/gen3/7dof/meshes/base_lin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 scale=1.15 1.15 1.15; visual mesh filename=package://kortex_description/arms/gen3/7dof/meshes/base_lin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
- link right_bota_link: geometry collision mesh filename=package://dual_arm_control_bringup/config/mounting.dae scale=0.001 0.001 0.001; visual mesh filename=package://dual_arm_control_bringup/config/mounting.dae scale=0.001 0.001 0.001
- link right_bracelet_link: geometry collision mesh filename=package://kortex_description/arms/gen3/7dof/meshes/bracelet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 scale=1.15 1.15 1.15; visual mesh filename=package://kortex_description/arms/gen3/7dof/meshes/bracelet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
- link right_forearm_link: geometry collision mesh filename=package://kortex_description/arms/gen3/7dof/meshes/forearm_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 scale=1.15 1.15 1.15; visual mesh filename=package://kortex_description/arms/gen3/7dof/meshes/forearm_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
- link right_half_arm_1_link: geometry collision mesh filename=package://kortex_description/arms/gen3/7dof/meshes/half_arm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 scale=1.15 1.15 1.15; visual mesh filename=package://kortex_description/arms/gen3/7dof/meshes/half_arm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
- link right_half_arm_2_link: geometry collision mesh filename=package://kortex_description/arms/gen3/7dof/meshes/half_arm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 scale=1.15 1.15 1.15; visual mesh filename=package://kortex_description/arms/gen3/7dof/meshes/half_arm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
- link right_robotiq_85_base_link: geometry collision mesh filename=package://dual_arm_control_bringup/config/robotiq_descripti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 scale=1.15 1.15 1.15; visual mesh filename=package://dual_arm_control_bringup/config/robotiq_descripti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
- link right_robotiq_85_left_finger_link: geometry collision mesh filename=package://dual_arm_control_bringup/config/robotiq_descripti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 scale=1.15 1.15 1.15; visual mesh filename=package://dual_arm_control_bringup/config/robotiq_descripti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
- link right_robotiq_85_left_finger_tip_link: geometry collision mesh filename=package://dual_arm_control_bringup/config/robotiq_descripti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 scale=1.15 1.15 1.15; visual mesh filename=package://dual_arm_control_bringup/config/robotiq_descripti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
- link right_robotiq_85_left_inner_knuckle_link: geometry collision mesh filename=package://dual_arm_control_bringup/config/robotiq_descripti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 scale=1.15 1.15 1.15; visual mesh filename=package://dual_arm_control_bringup/config/robotiq_descripti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
- link right_robotiq_85_left_knuckle_link: geometry collision mesh filename=package://dual_arm_control_bringup/config/robotiq_descripti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 scale=1.15 1.15 1.15; visual mesh filename=package://dual_arm_control_bringup/config/robotiq_descripti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
- link right_robotiq_85_right_finger_link: geometry collision mesh filename=package://dual_arm_control_bringup/config/robotiq_descripti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 scale=1.15 1.15 1.15; visual mesh filename=package://dual_arm_control_bringup/config/robotiq_descripti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
- link right_robotiq_85_right_finger_tip_link: geometry collision mesh filename=package://dual_arm_control_bringup/config/robotiq_descripti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 scale=1.15 1.15 1.15; visual mesh filename=package://dual_arm_control_bringup/config/robotiq_descripti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
- link right_robotiq_85_right_inner_knuckle_link: geometry collision mesh filename=package://dual_arm_control_bringup/config/robotiq_descripti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 scale=1.15 1.15 1.15; visual mesh filename=package://dual_arm_control_bringup/config/robotiq_descripti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
- link right_robotiq_85_right_knuckle_link: geometry collision mesh filename=package://dual_arm_control_bringup/config/robotiq_descripti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 scale=1.15 1.15 1.15; visual mesh filename=package://dual_arm_control_bringup/config/robotiq_descripti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
- link right_shoulder_link: geometry collision mesh filename=package://kortex_description/arms/gen3/7dof/meshes/shoulder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 scale=1.15 1.15 1.15; visual mesh filename=package://kortex_description/arms/gen3/7dof/meshes/shoulder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
- link right_spherical_wrist_1_link: geometry collision mesh filename=package://kortex_description/arms/gen3/7dof/meshes/spherica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 scale=1.15 1.15 1.15; visual mesh filename=package://kortex_description/arms/gen3/7dof/meshes/spherica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
- link right_spherical_wrist_2_link: geometry collision mesh filename=package://kortex_description/arms/gen3/7dof/meshes/spherica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 scale=1.15 1.15 1.15; visual mesh filename=package://kortex_description/arms/gen3/7dof/meshes/spherica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
